Commit message: mesh and world launch

File: urdf/udacity_bot.xacro (robot description, xacro)
@@ -209,5 +209,5 @@
       <origin xyz="0 0 0" rpy="0 0 0"/>
       <geometry>
-	<mesh filename="package://udacity_bot/meshes/hokuyo.dae"/>
+	<mesh filename="package://slam-simulation/meshes/hokuyo.dae"/>
       </geometry>
     </visual>

Commit message: migrating to a sane and maintained environment

File: urdf/udacity_bot.xacro (robot description, xacro)
@@ -17,5 +17,5 @@
           iyy="0.3" iyz="0"
           izz="0.3"
-      />
+	  />
     </inertial>
     <collision name='collision'>
@@ -85,5 +85,5 @@
           iyy="0.1" iyz="0"
           izz="0.1"
-      />
+	  />
     </inertial>
     <collision name='right_wheel_collision'>
@@ -127,5 +127,5 @@
           iyy="0.1" iyz="0"
           izz="0.1"
-      />
+	  />
     </inertial>
     <collision name='left_wheel_collision'>
@@ -160,5 +160,5 @@
     <joint_properties damping="1.0" friction="1.0"/>
   </joint>
-  <link name='camera'>
+  <link name='camera_link'>
     <pose>0 0 0 0 0 0</pose>
     <inertial>
@@ -169,10 +169,10 @@
           iyy="1e-6" iyz="0"
           izz="1e-6"
-      />
+	  />
     </inertial>
     <collision name='camera_collision'>
       <origin xyz="0 0 0" rpy="0 0 0"/>
       <geometry>
-	<box size="0.05 0.05 0.05"/>
+	<box size="0.02 0.02 0.02"/>
       </geometry>
     </collision>
@@ -180,5 +180,5 @@
       <origin xyz="0 0 0" rpy="0 0 0"/>
       <geometry>
-	<box size="0.05 0.05 0.05"/>
+	<box size="0.02 0.02 0.02"/>
       </geometry>
     </visual>
@@ -186,9 +186,9 @@
   <joint type="fixed" name="camera_joint">
     <origin xyz="0.2 0 0" rpy="0 0 0"/>
-    <child link="camera"/>
-    <parent link="chassis"/>
-  </joint>
-  <link name='hokuyo'>
-    <pose>0 0 0 0 0 0</pose>
+    <child link="camera_link"/>
+    <parent link="chassis"/>
+  </joint>
+  <link name='camera_rgbd_frame'>
+    <pose>0 0 0 -1.57 0 -1.57</pose>
     <inertial>
       <mass value="0.1"/>
@@ -198,5 +198,34 @@
           iyy="1e-6" iyz="0"
           izz="1e-6"
-      />
+	  />
+    </inertial>
+    <collision name='camera_rgb_collision'>
+      <origin xyz="0 0 0" rpy="0 0 0"/>
+      <geometry>
+	<box size="0.02 0.04 0.02"/>
+      </geometry>
+    </collision>
+    <visual name='camera_rgb_visual'>
+      <origin xyz="0 0 0" rpy="0 0 0"/>
+      <geometry>
+	<box size="0.02 0.04 0.02"/>
+      </geometry>
+    </visual>
+  </link>
+  <joint type="fixed" name="camera_rgb_joint">
+    <origin xyz="0.005 0 0.02" rpy="0 0 0"/>
+    <child link="camera_rgbd_frame"/>
+    <parent link="camera_link"/>
+  </joint>
+  <link name='hokuyo'>
+    <pose>0 0 0 0 0 0</pose>
+    <inertial>
+      <mass value="0.1"/>
+      <origin xyz="0.0 0 0" rpy="0 0 0"/>
+      <inertia
+          ixx="1e-6" ixy="0" ixz="0"
+          iyy="1e-6" iyz="0"
+          izz="1e-6"
+	  />
     </inertial>
     <collision name='hokuyo_collision'>

Commit message: working mapping and crime scene model world

File: urdf/udacity_bot.xacro (robot description, xacro)
@@ -163,5 +163,5 @@
     <pose>0 0 0 0 0 0</pose>
     <inertial>
-      <mass value="0.1"/>
+      <mass value="0"/>
       <origin xyz="0.0 0 0" rpy="0 0 0"/>
       <inertia
@@ -171,24 +171,12 @@
 	  />
     </inertial>
-    <collision name='camera_collision'>
-      <origin xyz="0 0 0" rpy="0 0 0"/>
-      <geometry>
-	<box size="0.02 0.02 0.02"/>
-      </geometry>
-    </collision>
-    <visual name='camera_visual'>
-      <origin xyz="0 0 0" rpy="0 0 0"/>
-      <geometry>
-	<box size="0.02 0.02 0.02"/>
-      </geometry>
-    </visual>
   </link>
   <joint type="fixed" name="camera_joint">
-    <origin xyz="0.2 0 0" rpy="0 0 0"/>
+    <origin xyz="0 0 0" rpy="-1.57 0 -1.57"/>
     <child link="camera_link"/>
     <parent link="chassis"/>
   </joint>
   <link name='camera_rgbd_frame'>
-    <pose>0 0 0 -1.57 0 -1.57</pose>
+    <pose>0 0 0 0 0 0</pose>
     <inertial>
       <mass value="0.1"/>
@@ -214,7 +202,7 @@
   </link>
   <joint type="fixed" name="camera_rgb_joint">
-    <origin xyz="0.005 0 0.02" rpy="0 0 0"/>
+    <origin xyz="0.2 0 0" rpy="0 0 0"/>
     <child link="camera_rgbd_frame"/>
-    <parent link="camera_link"/>
+    <parent link="chassis"/>
   </joint>
   <link name='hokuyo'>
